Commit message: fix STL naming

File: ROS2/reach_bravo_description_mk2/urdf/bravo_5.urdf.xacro (robot description, xacro)
@@ -14,5 +14,5 @@
             <visual>
                 <geometry>
-                    <mesh filename="package://reach_bravo_description_mk2/meshes/1019 A.stl"/>
+                    <mesh filename="package://reach_bravo_description_mk2/meshes/1019_A.stl"/>
                 </geometry>
                 <material name="bravo_black"/>
@@ -47,5 +47,5 @@
             <visual>
                 <geometry>
-                    <mesh filename="package://reach_bravo_description_mk2/meshes/1019 B.stl"/>
+                    <mesh filename="package://reach_bravo_description_mk2/meshes/1019_B.stl"/>
                 </geometry>
                 <origin xyz="0 0 0" rpy="0 0 3.14159"/>
@@ -61,5 +61,5 @@
             <visual>
                 <geometry>
-                    <mesh filename="package://reach_bravo_description_mk2/meshes/1013 A.stl"/>
+                    <mesh filename="package://reach_bravo_description_mk2/meshes/1013_A.stl"/>
                 </geometry>
                 <origin rpy="0 0 3.14159" xyz="0.0 00 0.0"/>
@@ -89,5 +89,5 @@
             <visual>
                 <geometry>
-                    <mesh filename="package://reach_bravo_description_mk2/meshes/1013 B.stl"/>
+                    <mesh filename="package://reach_bravo_description_mk2/meshes/1013_B.stl"/>
                 </geometry>
                 <material name="bravo_black"/>
@@ -121,5 +121,5 @@
             <visual>
                 <geometry>
-                    <mesh filename="package://reach_bravo_description_mk2/meshes/1023 A.stl"/>
+                    <mesh filename="package://reach_bravo_description_mk2/meshes/1023_A.stl"/>
                 </geometry>
                 <material name="bravo_black"/>
@@ -148,5 +148,5 @@
             <visual>
                 <geometry>
-                    <mesh filename="package://reach_bravo_description_mk2/meshes/1023 B.stl"/>
+                    <mesh filename="package://reach_bravo_description_mk2/meshes/1023_B.stl"/>
                 </geometry>
                 <material name="bravo_black"/>
@@ -188,5 +188,5 @@
             <visual>
                 <geometry>
-                    <mesh filename="package://reach_bravo_description_mk2/meshes/1023 C.stl"/>
+                    <mesh filename="package://reach_bravo_description_mk2/meshes/1023_C.stl"/>
                 </geometry>
                 <material name="bravo_black"/>

File: ROS2/reach_bravo_description_mk2/urdf/bravo_7.urdf.xacro (robot description, xacro)
@@ -14,5 +14,5 @@
             <visual>
                 <geometry>
-                    <mesh filename="package://reach_bravo_description_mk2/meshes/1019 A.stl"/>
+                    <mesh filename="package://reach_bravo_description_mk2/meshes/1019_A.stl"/>
                 </geometry>
                 <material name="bravo_black"/>
@@ -47,5 +47,5 @@
             <visual>
                 <geometry>
-                    <mesh filename="package://reach_bravo_description_mk2/meshes/1019 B.stl"/>
+                    <mesh filename="package://reach_bravo_description_mk2/meshes/1019_B.stl"/>
                 </geometry>
                 <origin xyz="0 0 0" rpy="0 0 3.14159"/>
@@ -61,5 +61,5 @@
             <visual>
                 <geometry>
-                    <mesh filename="package://reach_bravo_description_mk2/meshes/1013 A.stl"/>
+                    <mesh filename="package://reach_bravo_description_mk2/meshes/1013_A.stl"/>
                 </geometry>
                 <origin rpy="0 0 3.14159" xyz="0.0 00 0.0"/>
@@ -89,5 +89,5 @@
             <visual>
                 <geometry>
-                    <mesh filename="package://reach_bravo_description_mk2/meshes/1013 B.stl"/>
+                    <mesh filename="package://reach_bravo_description_mk2/meshes/1013_B.stl"/>
                 </geometry>
                 <material name="bravo_black"/>
@@ -121,5 +121,5 @@
             <visual>
                 <geometry>
-                    <mesh filename="package://reach_bravo_description_mk2/meshes/1026 A.stl"/>
+                    <mesh filename="package://reach_bravo_description_mk2/meshes/1026_A.stl"/>
                 </geometry>
                 <material name="bravo_black"/>
@@ -148,5 +148,5 @@
             <visual>
                 <geometry>
-                    <mesh filename="package://reach_bravo_description_mk2/meshes/1026 B.stl"/>
+                    <mesh filename="package://reach_bravo_description_mk2/meshes/1026_B.stl"/>
                 </geometry>
                 <material name="bravo_black"/>
@@ -188,5 +188,5 @@
             <visual>
                 <geometry>
-                    <mesh filename="package://reach_bravo_description_mk2/meshes/1026 C.stl"/>
+                    <mesh filename="package://reach_bravo_description_mk2/meshes/1026_C.stl"/>
                 </geometry>
                 <material name="bravo_black"/>
@@ -214,5 +214,5 @@
             <visual>
                 <geometry>
-                    <mesh filename="package://reach_bravo_description_mk2/meshes/1023 A.stl"/>
+                    <mesh filename="package://reach_bravo_description_mk2/meshes/1023_A.stl"/>
                 </geometry>
                 <material name="bravo_black"/>
@@ -241,5 +241,5 @@
             <visual>
                 <geometry>
-                    <mesh filename="package://reach_bravo_description_mk2/meshes/1023 B.stl"/>
+                    <mesh filename="package://reach_bravo_description_mk2/meshes/1023_B.stl"/>
                 </geometry>
                 <material name="bravo_black"/>
@@ -281,5 +281,5 @@
             <visual>
                 <geometry>
-                    <mesh filename="package://reach_bravo_description_mk2/meshes/1023 C.stl"/>
+                    <mesh filename="package://reach_bravo_description_mk2/meshes/1023_C.stl"/>
                 </geometry>
                 <material name="bravo_black"/>
